Commit message: Added the diamond shaped texture on the pads on the fingers, updated URDF and USD to fix the camera view mistake

File: dex1_d405_hand/dex1_1_d405.urdf (robot description, URDF)
Before this commit: robot dex1_1_d405, 10 links, 9 joints
Joints:
- joint d405_mount_to_optical: origin xyz=0.000000 0.058370 0.029108 rpy=0.523611 0.000000 0.000000 -> xyz=0.000000 0.058370 0.029108 rpy=-0.523611 0.000000 3.141593
